File: freeDSP-aurora-expansion-port-extender.kicad_sch (KiCad schematic)
At the start: 9 parts, among them J1 Conn_02x08_Odd_Even, J2 Conn_02x08_Odd_Even, J3 Conn_01x10, J4 Conn_01x10, U1 NCP1117-3.3_SOT223

Commit message: Update freeDSP-aurora-expansion-port-extender.kicad_sch
Other:
- note added: "C11 & C22 depends on the regulator U1"
Changed lines of the file:
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@@
     (stroke (width 0) (type solid))
+  )
+  (text "C11 & C22 depends on the regulator U1" (at 39.37 114.3 0)
+    (effects (font (size 1.27 1.27)) (justify left bottom))
   )
   (symbol (lib_id "Device:C") (at 36.068 91.186 0) (unit 1)
